File: circle/9axis/circle_9axis.brd (EAGLE design)
At the start: 10 x 10 mm, 9 parts

Commit message: Update circle
Parts:
- removed U$5: (no value), FaBo-etc:LOGO_OSHW_S
- moved U$3 6.20 mm to (5.38, 1.17)
Other:
- board text removed: "Rev. Beta9"
Changed lines of the file:
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@@
 <board>
 <plain>
-<text x="8.6" y="2.5" size="0.3" layer="21" rot="R180">Rev. Beta9</text>
 </plain>
 <attributes>
@@
 <element name="C2" library="FaBo-Capacitor" package="0402" value="0.1uf" x="1.524" y="3.2512"/>
 <element name="C1" library="FaBo-Capacitor" package="0402" value="1uf" x="8.5344" y="5.1054"/>
-<element name="U$3" library="FaBo" package="LOGO_FABO_S" value="" x="5.3816" y="7.3692"/>
-<element name="U$5" library="FaBo-etc" package="LOGO_OSHW_S" value="" x="5.3086" y="1.5494"/>
+<element name="U$3" library="FaBo" package="LOGO_FABO_S" value="" x="5.3816" y="1.1692"/>
 </elements>
 <signals>
