File: circle/color/circle_color.brd (EAGLE design)
At the start: 10 x 10 mm, 8 parts

Commit message: Update circle
Parts:
- removed C2: 0.1uf, FaBo-Capacitor:0402
- removed U$3: (no value), FaBo-etc:LOGO_FABO_S
- removed U1: (no value), FaBo-Sensor:VCNL4040M3OE
- added LED1: NSSW157T, FaBo-LED:NSSW157T
- added R3: (no value), FaBo-Resistors:0402
- added S1: HAMAMATSU-S11059, gclueSensor:HAMAMATSU-S11059
- U$2: value FABO-NANO -> (none); device FaBo-Template:FABO-NANO -> FaBo:LOGO_FABO_S
- U$4: value (none) -> FABO-NANO; device FaBo-etc:LOGO_OSHW_S -> FaBo-Template:FABO-NANO
- moved C1 7.33 mm to (1.24, 3.99)
- moved R1 6.88 mm to (8.71, 6.71)
- moved R2 6.84 mm to (8.69, 5.36)
- moved U$2 4.09 mm to (5.30, 1.00)
- moved U$4 3.07 mm to (5.08, 5.08)
Connections:
- removed net 3V3: C1.P$2, C2.P$2, R1.P$2, R2.P$2, U$2.VCC, U1.3, U1.4, U1.6
- new net +3V3: C1.P$2, R1.P$2, R2.P$2, S1.1, U$4.VCC
- new net N$2: LED1.CATHODE1, LED1.CATHODE2, R3.P$1
- net GND: now also R3.P$2, S1.2, S1.3, S1.4, S1.5, S1.7, S1.8, U$4.GND; no longer C2.P$1, U$2.GND, U1.1
- net N$1: now also LED1.ANODE1, LED1.ANODE2, U$4.2; no longer U1.2, U1.5
- net SCL: now also S1.6, U$4.0; no longer U$2.0, U1.8
- net SDA: now also S1.9, U$4.1; no longer U$2.1, U1.7
Routing:
- net +3V3: track 0.00 -> 25.9 mm, vias 0 -> 2
- net SCL: track 4.04 -> 21.1 mm, vias 1 -> 2
- net 3V3: track 16.7 -> 0.00 mm, vias 1 -> 0
- net GND: track 9.56 -> 24.3 mm, vias 1 -> 2
- net N$2: track 0.00 -> 14.3 mm, vias 0 -> 2
- net N$1: track 5.49 -> 15.8 mm, vias 0 -> 1
- net SDA: track 14.9 -> 8.21 mm, vias 1 -> 2
Other:
- board text added: "MADE IN JAPAN"
