File: circle/color/circle_color.sch (EAGLE design)
At the start: 5 parts

Commit message: Update circle
Parts:
- removed SI1145: SL-SI1145, FaBo-Mems:SL-SI1145
- removed U$2: FABO-NANO, FaBo-Template:FABO-NANO
- added LED1: NSSW157T, FaBo-LED:NSSW157T
- added R3: (no value), FaBo-Resistors:RESISTOR-0402
- added S1: HAMAMATSU-S11059, gclueSensor:HAMAMATSU-S11059
- added U$4: FABO-NANO, FaBo-Template:FABO-NANO
Connections:
- removed net 3V3: C1.2, R1.2, R2.2, SI1145.CVDD1, SI1145.CVDD2, SI1145.VDD, U$2.VCC
- new net +3V3: C1.2, R1.2, R2.2, S1.VDD, U$4.VCC
- new net N$1: LED1.ANODE, U$4.2
- new net N$2: LED1.CATHODE, R3.1
- net GND: now also R3.2, S1.GND1, S1.GND2, S1.GND3, S1.GND4, S1.GND5, S1.GND6, U$4.GND; no longer SI1145.GND, U$2.GND
- net SCL: now also R1.1, S1.SCL, U$4.0; no longer R2.1, SI1145.SCL, U$2.SCL
- net SDA: now also R2.1, S1.SDA, U$4.1; no longer R1.1, SI1145.SDA, U$2.SDA
Other:
- moved on the sheet: C1, R1, R2
