File: circle/humidity/circle_humidity.sch (EAGLE design)
At the start: 3 parts

Commit message: Update circle
Parts:
- removed U$2: FABO-NANO, FaBo-Template:FABO-NANO
- removed WS1: (no value), FaBo-LED:WS2818B
- added C2: 2.2pf, FaBo-Capacitor:CAPACITOR0402
- added LPC2985: (no value), FaBo-Supply:TI-LP2985-18DBVT
- added R1, R2: 4.7K, FaBo-Resistors:RESISTOR-0402
- added U$5: FABO-NANO, FaBo-Template:FABO-NANO
- added U$6: SILICONLABS-SI7034, FaBo-Mems:SILICONLABS-SI7034
- C1: value 0.1uf -> 1uf
Connections:
- removed net +5V: C1.2, U$2.VCC, WS1.VDD
- removed net DI_1: U$2.PIN-A, WS1.DIM
- removed net DO_1: WS1.DOUT
- new net 1.8V: C2.2, LPC2985.VOUT, R1.2, R2.2, U$6.VDD
- new net 3.3V: C1.2, LPC2985.ON/OFF, LPC2985.VIN, U$5.VCC
- new net SCL: R2.1, U$5.0, U$6.SCL
- new net SDA: R1.1, U$5.1, U$6.SDA
- net GND: now also C2.1, LPC2985.GND, U$5.GND, U$6.GND; no longer U$2.GND, WS1.VSS
Other:
- note added: "1.0.0"
- note removed: "1.0"
- moved on the sheet: C1
