File: circle/led/circle_color_led.brd (EAGLE design)
At the start: 10 x 10 mm, 3 parts

Commit message: Update circle
Parts:
- removed LED1: WS2818B, GClue-LED:WS2818B
- added U$3: (no value), FaBo:LOGO_FABO_S
- added WS1: (no value), FaBo-LED:WS2818B
- C1: device GClue-Capacitor:0603 -> FaBo-Capacitor:0402
- moved C1 5.39 mm to (1.27, 5.08)
Connections:
- net +5V: now also C1.P$2, WS1.1; no longer C1.2, LED1.1
- net DI_1: now also WS1.4; no longer LED1.4
- net DO_1: now also WS1.2; no longer LED1.2
- net GND: now also C1.P$1, WS1.3; no longer C1.1, LED1.3
Routing:
- net GND: track 17.0 -> 10.8 mm
- net +5V: track 9.10 -> 6.43 mm
Changed lines of the file:
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@@
 <setting verticaltext="up"/>
 </settings>
-<grid distance="0.05" unitdist="inch" unit="inch" style="lines" multiple="1" display="no" altdistance="0.025" altunitdist="inch" altunit="inch"/>
+<grid distance="0.1" unitdist="inch" unit="inch" style="lines" multiple="1" display="no" altdistance="0.025" altunitdist="inch" altunit="inch"/>
 <layers>
 <layer number="1" name="Top" color="4" fill="1" visible="yes" active="yes"/>
@@
 </autorouter>
 <elements>
-<element name="C1" library="GClue-Capacitor" package="0603" value="0.1uf" x="5.08" y="1.27"/>
-<element name="LED1" library="GClue-LED" package="WS2818B" value="WS2818B" x="5.08" y="5.08"/>
 <element name="U$2" library="FaBo-Template" package="FABO-NANO" value="FABO-NANO" x="5.08" y="5.08"/>
+<element name="WS1" library="FaBo-LED" package="WS2818B" value="" x="5.08" y="5.334"/>
+<element name="C1" library="FaBo-Capacitor" package="0402" value="0.1uf" x="1.27" y="5.08"/>
+<element name="U$3" library="FaBo" package="LOGO_FABO_S" value="" x="5.334" y="0.762"/>
 </elements>
 <signals>
 <signal name="GND">
 <contactref element="U$2" pad="GND"/>
-<contactref element="C1" pad="1"/>
-<contactref element="LED1" pad="3"/>
-<wire x1="4.2672" y1="3.5052" x2="4.2672" y2="1.3716" width="0.1524" layer="1"/>
-<wire x1="1.524" y1="6.2484" x2="4.2672" y2="3.5052" width="0.1524" layer="1"/>
-<wire x1="1.524" y1="7.3152" x2="1.524" y2="6.2484" width="0.1524" layer="1"/>
-<wire x1="1.6764" y1="7.4676" x2="1.524" y2="7.3152" width="0.1524" layer="1"/>
-<wire x1="3.5052" y1="7.4676" x2="1.6764" y2="7.4676" width="0.1524" layer="1"/>
-<wire x1="7.4676" y1="3.5052" x2="5.4864" y2="5.4864" width="0.1524" layer="1"/>
-<wire x1="5.4864" y1="5.4864" x2="3.5052" y2="7.4676" width="0.1524" layer="1"/>
-<wire x1="4.2672" y1="1.3716" x2="4.33" y2="1.27" width="0.1524" layer="1"/>
-<wire x1="7.4676" y1="3.5052" x2="7.58" y2="3.38" width="0.1524" layer="1"/>
-<wire x1="6.2484" y1="6.2484" x2="6.2484" y2="7.0104" width="0.1524" layer="16"/>
-<wire x1="5.4864" y1="5.4864" x2="6.2484" y2="6.2484" width="0.1524" layer="16"/>
-<wire x1="6.2484" y1="7.0104" x2="6.35" y2="7.08" width="0.1524" layer="16"/>
-<via x="5.4864" y="5.4864" extent="1-16" drill="0.3048"/>
+<contactref element="WS1" pad="3"/>
+<contactref element="C1" pad="P$1"/>
+<wire x1="1.524" y1="4.4196" x2="0.9144" y2="5.0292" width="0.1524" layer="1"/>
+<wire x1="4.7244" y1="4.4196" x2="1.524" y2="4.4196" width="0.1524" layer="1"/>
+<wire x1="5.4864" y1="3.6576" x2="4.7244" y2="4.4196" width="0.1524" layer="1"/>
+<wire x1="7.4676" y1="3.6576" x2="6.4008" y2="3.6576" width="0.1524" layer="1"/>
+<wire x1="6.4008" y1="3.6576" x2="5.4864" y2="3.6576" width="0.1524" layer="1"/>
+<wire x1="0.9144" y1="5.0292" x2="0.81" y2="5.08" width="0.1524" layer="1"/>
+<wire x1="7.4676" y1="3.6576" x2="7.58" y2="3.634" width="0.1524" layer="1"/>
+<wire x1="6.4008" y1="4.572" x2="6.4008" y2="7.0104" width="0.1524" layer="16"/>
+<wire x1="6.4008" y1="3.6576" x2="6.4008" y2="4.572" width="0.1524" layer="1"/>
+<wire x1="6.4008" y1="7.0104" x2="6.35" y2="7.08" width="0.1524" layer="16"/>
+<via x="6.4008" y="4.572" extent="1-16" drill="0.3048"/>
 <polygon width="0.4064" layer="1">
 <vertex x="0" y="0"/>
@@
 <signal name="+5V">
 <contactref element="U$2" pad="VCC"/>
-<contactref element="LED1" pad="1"/>
-<contactref element="C1" pad="2"/>
-<wire x1="5.7912" y1="3.5052" x2="5.7912" y2="1.3716" width="0.1524" layer="1"/>
-<wire x1="2.5908" y1="6.7056" x2="3.9624" y2="5.334" width="0.1524" layer="1"/>
-<wire x1="3.9624" y1="5.334" x2="5.7912" y2="3.5052" width="0.1524" layer="1"/>
-<wire x1="5.7912" y1="1.3716" x2="5.83" y2="1.27" width="0.1524" layer="1"/>
-<wire x1="2.5908" y1="6.7056" x2="2.58" y2="6.78" width="0.1524" layer="1"/>
-<wire x1="5.0292" y1="6.4008" x2="5.0292" y2="7.0104" width="0.1524" layer="16"/>
-<wire x1="3.9624" y1="5.334" x2="5.0292" y2="6.4008" width="0.1524" layer="16"/>
-<wire x1="5.0292" y1="7.0104" x2="5.15" y2="7.08" width="0.1524" layer="16"/>
-<via x="3.9624" y="5.334" extent="1-16" drill="0.3048"/>
+<contactref element="WS1" pad="1"/>
+<contactref element="C1" pad="P$2"/>
+<wire x1="1.8288" y1="6.4008" x2="1.8288" y2="5.7912" width="0.1524" layer="1"/>
+<wire x1="1.8288" y1="5.7912" x2="1.8288" y2="5.1816" width="0.1524" layer="1"/>
+<wire x1="2.4384" y1="7.0104" x2="1.8288" y2="6.4008" width="0.1524" layer="1"/>
+<wire x1="1.8288" y1="5.1816" x2="1.73" y2="5.08" width="0.1524" layer="1"/>
+<wire x1="2.4384" y1="7.0104" x2="2.58" y2="7.034" width="0.1524" layer="1"/>
+<wire x1="3.048" y1="5.7912" x2="1.8288" y2="5.7912" width="0.1524" layer="1"/>
+<wire x1="4.2672" y1="5.7912" x2="3.048" y2="5.7912" width="0.1524" layer="16"/>
+<wire x1="5.0292" y1="6.5532" x2="4.2672" y2="5.7912" width="0.1524" layer="16"/>
+<wire x1="5.0292" y1="7.0104" x2="5.0292" y2="6.5532" width="0.1524" layer="16"/>
+<wire x1="5.0292" y1="7.0104" x2="5.08" y2="7.08" width="0.1524" layer="16"/>
+<via x="3.048" y="5.7912" extent="1-16" drill="0.3048"/>
+</signal>
+<signal name="DI_1">
+<contactref element="U$2" pad="2"/>
+<contactref element="WS1" pad="4"/>
+<wire x1="5.1816" y1="4.7244" x2="7.4676" y2="7.0104" width="0.1524" layer="1"/>
+<wire x1="5.1816" y1="3.2004" x2="5.1816" y2="4.7244" width="0.1524" layer="16"/>
+<wire x1="7.4676" y1="7.0104" x2="7.58" y2="7.034" width="0.1524" layer="1"/>
+<wire x1="5.1816" y1="3.2004" x2="5.08" y2="3.08" width="0.1524" layer="16"/>
+<via x="5.1816" y="4.7244" extent="1-16" drill="0.3048"/>
 </signal>
 <signal name="DO_1">
-<contactref element="LED1" pad="2"/>
-</signal>
-<signal name="DI_1">
-<contactref element="LED1" pad="4"/>
-<contactref element="U$2" pad="2"/>
-<wire x1="6.2484" y1="5.4864" x2="7.4676" y2="6.7056" width="0.1524" layer="1"/>
-<wire x1="6.2484" y1="4.7244" x2="6.2484" y2="5.4864" width="0.1524" layer="16"/>
-<wire x1="5.1816" y1="3.6576" x2="6.2484" y2="4.7244" width="0.1524" layer="16"/>
-<wire x1="5.1816" y1="3.2004" x2="5.1816" y2="3.6576" width="0.1524" layer="16"/>
-<wire x1="7.4676" y1="6.7056" x2="7.58" y2="6.78" width="0.1524" layer="1"/>
-<wire x1="5.1816" y1="3.2004" x2="5.15" y2="3.13" width="0.1524" layer="16"/>
-<via x="6.2484" y="5.4864" extent="1-16" drill="0.3048"/>
+<contactref element="WS1" pad="2"/>
 </signal>
 </signals>
