File: circle/proximinity/circle_proximity.brd (EAGLE design)
At the start: 10 x 10 mm, 8 parts

Commit message: Update circle
Parts:
- removed U$4: (no value), FaBo-etc:LOGO_OSHW_S
- moved U$3 6.00 mm to (5.26, 1.19)
Changed lines of the file:
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@@
 <element name="C1" library="FaBo-Capacitor" package="0402" value="0.1uf" x="8.382" y="5.6642"/>
 <element name="C2" library="FaBo-Capacitor" package="0402" value="0.1uf" x="8.3566" y="4.5212"/>
-<element name="U$3" library="FaBo-etc" package="LOGO_FABO_S" value="" x="5.2578" y="7.1882"/>
-<element name="U$4" library="FaBo-etc" package="LOGO_OSHW_S" value="" x="5.1308" y="2.0066"/>
+<element name="U$3" library="FaBo-etc" package="LOGO_FABO_S" value="" x="5.2578" y="1.1882"/>
 </elements>
 <signals>
